File: SingleWaterTimer.kicad_sch (KiCad schematic)
At the start: 15 parts, among them J1 Conn_01x02_Pin, J2 230VAC, J3 PUMP, J4 Conn_01x07_Pin, K1 SCHRACK V23061A1005A302, Q1 PN2222A, SW2 RotaryEncoder_Switch_MP, U1 L7805

Commit message: schemas
Connections:
- net Rotat1: now also UESP32-C3-EH1.2 (A2)
- net SW: now also UESP32-C3-EH1.4 (A4-SCK)
- net rotat2: now also UESP32-C3-EH1.3 (A3)
Other:
- moved on the sheet: D1, J2, J3, K1, Q1
